File: driver1.kicad_sch (KiCad schematic)
At the start: 91 parts, among them J1 FB CT, J2 GDT, J3 24VDC INPUT, SW1 PHASE, SW2 SKIP_ENABLE, U1 IX4340, U10 L7809, U11 L7805, U12 74AHC1G08, U13 74AHC158, U2 MCP6567, U3 74AHC74, U4 IF-D95T, U5 74AHC14, U6 TLV3501AID, U8 AOD609, U9 AOD609

Commit message: Fix footprint link
Parts:
- U4: footprint IF parts:IF-D95T_IFB -> footprints:IF-D95T_IFB
Changed lines of the file:
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@@
 	)
 	(symbol
-		(lib_id "2026-03-23_09-37-43:IF-D95T")
-		(at 163.83 158.75 0)
-		(unit 1)
-		(exclude_from_sim no)
-		(in_bom yes)
-		(on_board yes)
-		(dnp no)
-		(fields_autoplaced yes)
-		(property "Reference" "U4"
-			(at 163.83 148.59 0)
-			(effects
-				(font
-					(size 1.524 1.524)
-				)
-			)
-		)
-		(property "Value" "IF-D95T"
-			(at 163.83 151.13 0)
-			(effects
-				(font
-					(size 1.524 1.524)
-				)
-			)
-		)
-		(property "Footprint" "IF parts:IF-D95T_IFB"
-			(at 154.94 153.67 0)
-			(effects
-				(font
-					(size 1.27 1.27)
-					(italic yes)
-				)
-				(hide yes)
-			)
-		)
-		(property "Datasheet" "IF-D95T"
-			(at 154.94 153.67 0)
-			(effects
-				(font
-					(size 1.27 1.27)
-					(italic yes)
-				)
-				(hide yes)
-			)
-		)
-		(property "Description" ""
-			(at 154.94 153.67 0)
-			(effects
-				(font
-					(size 1.27 1.27)
-				)
-				(hide yes)
-			)
-		)
-		(pin "1"
-		)
-		(pin "2"
-		)
-		(pin "3"
-		)
-		(instances
-			(project "driver1"
-				(path "/ed4ed053-ef94-4597-a27c-c8d8624d8bb7"
-					(reference "U4")
-					(unit 1)
-				)
-			)
-		)
-	)
-	(symbol
 		(lib_id "power:+12V")
 		(at 325.12 74.93 0)
@@
 				)
 			)
+		)
+	)
+	(symbol
+		(lib_id "2026-03-23_09-37-43:IF-D95T")
+		(at 163.83 158.75 0)
+		(unit 1)
+		(exclude_from_sim no)
+		(in_bom yes)
+		(on_board yes)
+		(dnp no)
+		(fields_autoplaced yes)
+		(property "Reference" "U4"
+			(at 163.83 148.59 0)
+			(effects
+				(font
+					(size 1.524 1.524)
+				)
+			)
+		)
+		(property "Value" "IF-D95T"
+			(at 163.83 151.13 0)
+			(effects
+				(font
+					(size 1.524 1.524)
+				)
+			)
+		)
+		(property "Footprint" "footprints:IF-D95T_IFB"
+			(at 154.94 153.67 0)
+			(effects
+				(font
+					(size 1.27 1.27)
+					(italic yes)
+				)
+				(hide yes)
+			)
+		)
+		(property "Datasheet" "IF-D95T"
+			(at 154.94 153.67 0)
+			(effects
+				(font
+					(size 1.27 1.27)
+					(italic yes)
+				)
+				(hide yes)
+			)
+		)
+		(property "Description" ""
+			(at 154.94 153.67 0)
+			(effects
+				(font
+					(size 1.27 1.27)
+				)
+				(hide yes)
+			)
+		)
+		(pin "3"
+		)
+		(pin "2"
+		)
+		(pin "1"
+		)
+		(instances
+			(project ""
+				(path "/ed4ed053-ef94-4597-a27c-c8d8624d8bb7"
+					(reference "U4")
+					(unit 1)
+				)
+			)

Commit message: Progress
Parts:
- removed SW1: PHASE, symbol Switch:SW_SPST
- removed SW2: SKIP_ENABLE, symbol Switch:SW_SPDT
- removed U6: TLV3501AID, Package_SO:SOIC-8_3.9x4.9mm_P1.27mm, symbol Comparator:TLV3501AID
- added J4: MODE, symbol Connector:Conn_01x03_Pin
- added J5: PHASE, symbol Connector:Conn_01x02_Pin
- added R23: 10k, Resistor_SMD:R_0603_1608Metric_Pad0.98x0.95mm_HandSolder, symbol Device:R
- added U7: TLV3501AIDBV, Package_TO_SOT_SMD:SOT-23-6, symbol Comparator:TLV3501AIDBV
- C11, C12, C13, C14, C15, C6: footprint Capacitor_SMD:C_0603_1608Metric_Pad1.08x0.95mm_HandSolder -> Capacitor_SMD:C_0805_2012Metric_Pad1.18x1.45mm_HandSolder
- C16, C17: footprint Capacitor_SMD:C_0603_1608Metric_Pad1.08x0.95mm_HandSolder -> Capacitor_SMD:C_1210_3225Metric_Pad1.33x2.70mm_HandSolder
- R1: footprint Resistor_SMD:R_0603_1608Metric_Pad0.98x0.95mm_HandSolder -> Resistor_SMD:R_2512_6332Metric_Pad1.40x3.35mm_HandSolder
- R18, R2: footprint Resistor_SMD:R_0603_1608Metric_Pad0.98x0.95mm_HandSolder -> Resistor_SMD:R_1210_3225Metric_Pad1.30x2.65mm_HandSolder
- U13: footprint (none) -> Package_SO:TSSOP-16_4.4x5mm_P0.65mm
Connections:
- net +5V: now also U7.4 (V+)
- net FB: now also J4.3 (Pin_3), U7.5
- net GND: now also J5.2 (Pin_2), R23.2, U7.2 (V-), U7.6 (SHDN)
- net INTERRUPTER: now also J4.1 (Pin_1)
- net at R22.2, U13.3 (I1a), U13.5 (I0b)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: now also J5.1 (Pin_1)
- net at R4.1, R5.1, R6.2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: now also U7.3 (+)
- net at C2.2, R8.1: now also U7.1 (-)
- net at U3.3 (C): now also J4.2 (Pin_2), R23.1
Other:
- moved on the sheet: C18, C19, C20, C21, C22, C23, C24, C25, D6, D7, J3, U10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

Commit message: progress
Parts:
- removed H1, H2, H3, H4: MountingHole, MountingHole:MountingHole_3.2mm_M3, symbol Mechanical:MountingHole
- added H1, H2, H3, H4: MountingHole_Pad, MountingHole:MountingHole_3.2mm_M3_Pad, symbol Mechanical:MountingHole_Pad
- J3: renamed from J4; footprint (none) -> Connector_PinHeader_2.54mm:PinHeader_1x03_P2.54mm_Vertical_SMD_Pin1Left
- J4: renamed from J5; footprint (none) -> Connector_PinHeader_2.54mm:PinHeader_1x02_P2.54mm_Vertical_SMD_Pin1Left
- RV1: footprint Potentiometer_THT:Potentiometer_Bourns_3339P_Vertical -> Potentiometer_THT:Potentiometer_Bourns_3296W_Vertical
- U6: renamed from U5; footprint (none) -> Package_SO:TSSOP-14_4.4x5mm_P0.65mm
- U7: renamed from U3; footprint (none) -> Package_SO:TSSOP-14_4.4x5mm_P0.65mm
- U8: renamed from U12; footprint (none) -> Package_TO_SOT_SMD:SOT-353_SC-70-5
- U9: renamed from U1; footprint (none) -> Package_SO:SOIC-8-1EP_3.9x4.9mm_P1.27mm_EP2.29x3mm
- renumbered C2 to C10, C23 to C11, C3 to C12, C24 to C14, C25 to C15, C26 to C16, C9 to C17, C27 to C18, C28 to C19, C19 to C2, C10 to C20, C11 to C21, C6 to C22, C13 to C23, C14 to C24, C12 to C25, C15 to C26, C4 to C27, C16 to C28, C17 to C29, C8 to C3, C18 to C4, C20 to C5, C5 to C6, C22 to C8, C21 to C9, D2 to D1, D5 to D10, D6 to D2, D1 to D3, D7 to D4, D8 to D5, D9 to D6, D10 to D7, D3 to D8, D4 to D9, J3 to J2, J2 to J5, R4 to R10, R8 to R11, R5 to R12, R15 to R13, R19 to R14, R20 to R15, R21 to R16, R23 to R17, R11 to R18, R16 to R19, R22 to R20, R12 to R21, R17 to R22, R18 to R23, R9 to R3, R13 to R4, R14 to R5, R3 to R6, R10 to R7, R6 to R8, R7 to R9, RV4 to RV2, RV2 to RV4, TP2 to TP1, TP3 to TP2, TP1 to TP3, U10 to U1, U8 to U10, U9 to U11, U13 to U12, U7 to U3, U11 to U4, U4 to U5
Connections:
- net GND: now also U9.9 (EP)
- no-connect marks 4 -> 8

Commit message: pcb progress
Parts:
- J3: footprint Connector_PinHeader_2.54mm:PinHeader_1x03_P2.54mm_Vertical_SMD_Pin1Left -> Connector_PinHeader_2.54mm:PinHeader_1x03_P2.54mm_Vertical
- J4: footprint Connector_PinHeader_2.54mm:PinHeader_1x02_P2.54mm_Vertical_SMD_Pin1Left -> Connector_PinHeader_2.54mm:PinHeader_1x02_P2.54mm_Vertical
- U9: footprint Package_SO:SOIC-8-1EP_3.9x4.9mm_P1.27mm_EP2.29x3mm -> Package_SO:SOIC-8_3.9x4.9mm_P1.27mm
Connections:
- net A: now also U12.12 (Zc); no longer U12.4 (Za)
- net B: now also U12.9 (Zd); no longer U12.7 (Zb)
- net GND: now also U12.2 (I0a), U12.3 (I1a), U12.5 (I0b), U12.6 (I1b), U6.9; no longer U12.10 (I1d), U12.11 (I0d), U12.13 (I1c), U12.14 (I0c), U6.13, U9.9 (EP)
- net INTERRUPTER: now also U6.4, U8.2; no longer U6.6, U8.1
- net INTERRUPTER_LED: now also U6.6; no longer U6.8
- net ~{RESET}: now also U6.12; no longer U6.2
- net at C24.1, D10.2 (A), R22.2: now also U10.5 (G2); no longer U11.5 (G2)
- net at J4.1 (Pin_1), R20.2, U6.11: now also U12.11 (I0d), U12.13 (I1c); no longer U12.3 (I1a), U12.5 (I0b)
- net at J5.2 (Pin_2): now also U10.3 (D); no longer U11.3 (D)
- net at C22.2, D8.1 (K), R19.1: now also U6.13; no longer U6.1
- net at C23.1, D9.2 (A), R21.2: now also U11.5 (G2); no longer U10.5 (G2)
- net at C23.2, U9.7 (OUTA): now also U11.2 (G1); no longer U10.2 (G1)
- net at C28.1, R23.1: now also U11.3 (D); no longer U10.3 (D)
- net at U7.6 (~{Q}): now also U8.1; no longer U8.2
- net at C24.2, U9.5 (OUTB): now also U10.2 (G1); no longer U11.2 (G1)
- net at R13.1, U5.2 (OUTPUT): now also U6.1; no longer U6.3
- new net: U12.10 (I1d), U12.14 (I0c), U6.10
- new net: U6.2, U6.3, U6.5
Other:
- moved on the sheet: J3, R17, R18, U10, U11, U6A, U6B, U6C, U7A

Commit message: baby steps
Parts:
- removed TP4: UVLO_out, TestPoint:TestPoint_Pad_D2.0mm, symbol Connector:TestPoint
Connections:
- net +5V: now also D5.2 (A); no longer R14.1
- net GND: now also J1.2 (Pin_2), R14.2, R15.2, R16.2; no longer D5.1 (K), D6.1 (K), D7.1 (K), J1.1 (Pin_1)
- net INTERRUPTER_LED: now also D6.2 (A); no longer R15.1
- net SKIP_LED: now also D7.2 (A); no longer R16.1
- net at C1.1, R1.2, RV1.1: now also J1.1 (Pin_1); no longer J1.2 (Pin_2)
- new net: D5.1 (K), R14.1
- new net: D6.1 (K), R15.1
- new net: D7.1 (K), R16.1
Other:
- moved on the sheet: D5, D6, D7, J1, R14, R15, R16
Changed lines of the file:
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@@
 		(color 0 0 0 0)
 	)
-	(junction
-		(at 106.68 204.47)
-		(diameter 0)
-		(color 0 0 0 0)
-	)
 	(no_connect
 		(at 367.03 34.29)
@@
 	(wire
 		(pts
+			(xy 25.4 97.79) (xy 26.67 97.79)
+		)
+		(stroke
+			(width 0)
+			(type default)
+		)
+	)
+	(wire
+		(pts
 			(xy 134.62 44.45) (xy 134.62 46.99)
 		)
@@
 	(wire
 		(pts
-			(xy 25.4 97.79) (xy 26.67 97.79)
-		)
-		(stroke
-			(width 0)
-			(type default)
-		)
-	)
-	(wire
-		(pts
 			(xy 45.72 201.93) (xy 59.69 201.93)
 		)
@@
 	(wire
 		(pts
-			(xy 106.68 204.47) (xy 107.95 204.47)
-		)
-		(stroke
-			(width 0)
-			(type default)
-		)
-	)
-	(wire
-		(pts
 			(xy 229.87 22.86) (xy 238.76 22.86)
 		)
@@
 	(wire
 		(pts
-			(xy 105.41 204.47) (xy 106.68 204.47)
+			(xy 105.41 204.47) (xy 107.95 204.47)
 		)
 		(stroke
@@
 	(wire
 		(pts
-			(xy 106.68 198.12) (xy 106.68 204.47)
-		)
-		(stroke
-			(width 0)
-			(type default)
-		)
-	)
-	(wire
-		(pts
 			(xy 182.88 151.13) (xy 181.61 151.13)
 		)
@@
 	(symbol
 		(lib_id "Device:R")
-		(at 198.12 194.31 90)
+		(at 208.28 194.31 90)
 		(unit 1)
 		(body_style 1)
@@
 		(dnp no)
 		(property "Reference" "R14"
-			(at 198.12 189.484 90)
+			(at 208.28 189.484 90)
 			(show_name no)
 			(do_not_autoplace no)
@@
 		)
 		(property "Value" "470R"
-			(at 198.12 192.024 90)
+			(at 208.28 192.024 90)
 			(show_name no)
 			(do_not_autoplace no)
@@
 		)
 		(property "Footprint" "Resistor_SMD:R_0603_1608Metric_Pad0.98x0.95mm_HandSolder"
-			(at 198.12 196.088 90)
+			(at 208.28 196.088 90)
 			(hide yes)
 			(show_name no)
@@
 		)
 		(property "Datasheet" ""
-			(at 198.12 194.31 0)
+			(at 208.28 194.31 0)
 			(hide yes)
 			(show_name no)
@@
 		)
 		(property "Description" "Resistor"
-			(at 198.12 194.31 0)
+			(at 208.28 194.31 0)
 			(hide yes)
 			(show_name no)
@@
 	)
 	(symbol
-		(lib_id "Connector:TestPoint")
-		(at 106.68 198.12 0)
-		(unit 1)
-		(body_style 1)
-		(exclude_from_sim no)
-		(in_bom yes)
-		(on_board yes)
-		(in_pos_files yes)
-		(dnp no)
-		(fields_autoplaced yes)
-		(property "Reference" "TP4"
-			(at 109.22 193.5479 0)
-			(show_name no)
-			(do_not_autoplace no)
-			(effects
-				(font
-					(size 1.27 1.27)
-				)
-				(justify left)
-			)
-		)
-		(property "Value" "UVLO_out"
-			(at 109.22 196.0879 0)
-			(show_name no)
-			(do_not_autoplace no)
-			(effects
-				(font
-					(size 1.27 1.27)
-				)
-				(justify left)
-			)
-		)
-		(property "Footprint" "TestPoint:TestPoint_Pad_D2.0mm"
-			(at 111.76 198.12 0)
-			(hide yes)
-			(show_name no)
-			(do_not_autoplace no)
-			(effects
-				(font
-					(size 1.27 1.27)
-				)
-			)
-		)
-		(property "Datasheet" ""
-			(at 111.76 198.12 0)
-			(hide yes)
-			(show_name no)
-			(do_not_autoplace no)
-			(effects
-				(font
-					(size 1.27 1.27)
-				)
-			)
-		)
-		(property "Description" "test point"
-			(at 106.68 198.12 0)
-			(hide yes)
-			(show_name no)
-			(do_not_autoplace no)
-			(effects
-				(font
-					(size 1.27 1.27)
-				)
-			)
-		)
-		(pin "1"
-		)
-		(instances
-			(project "driver1"
-				(path "/ed4ed053-ef94-4597-a27c-c8d8624d8bb7"
-					(reference "TP4")
-					(unit 1)
-				)
-			)
-		)
-	)
-	(symbol
 		(lib_id "power:+24V")
 		(at 50.8 26.67 0)
@@
 	(symbol
 		(lib_id "Device:LED")
-		(at 208.28 205.74 180)
+		(at 198.12 205.74 180)
 		(unit 1)
 		(body_style 1)
@@
 		(dnp no)
 		(property "Reference" "D6"
-			(at 208.28 199.644 0)
+			(at 198.12 199.644 0)
 			(show_name no)
 			(do_not_autoplace no)
@@
 		)
 		(property "Value" "INTERRUPTER"
-			(at 208.28 202.184 0)
+			(at 198.12 202.184 0)
 			(show_name no)
 			(do_not_autoplace no)
@@
 		)
 		(property "Footprint" "LED_THT:LED_D5.0mm"
-			(at 208.28 205.74 0)
+			(at 198.12 205.74 0)
 			(hide yes)
 			(show_name no)
@@
 		)
 		(property "Datasheet" ""
-			(at 208.28 205.74 0)
+			(at 198.12 205.74 0)
 			(hide yes)
 			(show_name no)
@@
 		)
 		(property "Description" "Light emitting diode"
-			(at 208.28 205.74 0)
+			(at 198.12 205.74 0)
 			(hide yes)
 			(show_name no)
@@
 		)
 		(property "Sim.Pins" "1=K 2=A"
-			(at 208.28 205.74 0)
+			(at 198.12 205.74 0)
 			(hide yes)
 			(show_name no)
@@
 	(symbol
 		(lib_id "Device:LED")
-		(at 208.28 194.31 180)
+		(at 198.12 194.31 180)
 		(unit 1)
 		(body_style 1)
@@
 		(dnp no)
 		(property "Reference" "D5"
-			(at 208.28 188.468 0)
+			(at 198.12 188.468 0)
 			(show_name no)
 			(do_not_autoplace no)
@@
 		)
 		(property "Value" "5V_OK"
-			(at 208.28 191.008 0)
+			(at 198.12 191.008 0)
 			(show_name no)
 			(do_not_autoplace no)
@@
 		)
 		(property "Footprint" "LED_THT:LED_D5.0mm"
-			(at 208.28 194.31 0)
+			(at 198.12 194.31 0)
 			(hide yes)
 			(show_name no)
@@
 		)
 		(property "Datasheet" ""
-			(at 208.28 194.31 0)
+			(at 198.12 194.31 0)
 			(hide yes)
 			(show_name no)
@@
 		)
 		(property "Description" "Light emitting diode"
-			(at 208.28 194.31 0)
+			(at 198.12 194.31 0)
 			(hide yes)
 			(show_name no)
@@
 		)
 		(property "Sim.Pins" "1=K 2=A"
-			(at 208.28 194.31 0)
+			(at 198.12 194.31 0)
 			(hide yes)
 			(show_name no)
@@
 	(symbol
 		(lib_id "Device:LED")
-		(at 208.28 215.9 180)
+		(at 198.12 215.9 180)
 		(unit 1)
 		(body_style 1)
@@
 		(dnp no)
 		(property "Reference" "D7"
-			(at 208.28 210.566 0)
+			(at 198.12 210.566 0)
 			(show_name no)
 			(do_not_autoplace no)
@@
 		)
 		(property "Value" "SKIP"
-			(at 208.28 213.106 0)
+			(at 198.12 213.106 0)
 			(show_name no)
 			(do_not_autoplace no)
@@
 		)
 		(property "Footprint" "LED_THT:LED_D5.0mm"
-			(at 208.28 215.9 0)
+			(at 198.12 215.9 0)
 			(hide yes)
 			(show_name no)
@@
 		)
 		(property "Datasheet" ""
-			(at 208.28 215.9 0)
+			(at 198.12 215.9 0)
 			(hide yes)
 			(show_name no)
@@
 		)
 		(property "Description" "Light emitting diode"
-			(at 208.28 215.9 0)
+			(at 198.12 215.9 0)
 			(hide yes)
 			(show_name no)
@@
 		)
 		(property "Sim.Pins" "1=K 2=A"
-			(at 208.28 215.9 0)
+			(at 198.12 215.9 0)
 			(hide yes)
 			(show_name no)
@@
 	(symbol
 		(lib_id "Connector:Screw_Terminal_01x02")
-		(at 20.32 97.79 180)
+		(at 20.32 95.25 0)
+		(mirror y)
 		(unit 1)
 		(body_style 1)
@@
 		(in_pos_files yes)
 		(dnp no)
-		(fields_autoplaced yes)
 		(property "Reference" "J1"
-			(at 20.32 88.9 0)
+			(at 20.32 104.14 0)
 			(show_name no)
 			(do_not_autoplace no)
@@
 		)
 		(property "Value" "FB CT"
-			(at 20.32 91.44 0)
+			(at 20.32 101.6 0)
 			(show_name no)
 			(do_not_autoplace no)
@@
 		)
 		(property "Footprint" "TerminalBlock_Altech:Altech_AK100_1x02_P5.00mm"
-			(at 20.32 97.79 0)
+			(at 20.32 95.25 0)
 			(hide yes)
 			(show_name no)
@@
 		)
 		(property "Datasheet" ""
-			(at 20.32 97.79 0)
+			(at 20.32 95.25 0)
 			(hide yes)
 			(show_name no)
@@
 		)
 		(property "Description" "Generic screw terminal, single row, 01x02, script generated (kicad-library-utils/schlib/autogen/connector/)"
-			(at 20.32 97.79 0)
+			(at 20.32 95.25 0)
 			(hide yes)
 			(show_name no)
@@
 	(symbol
 		(lib_id "Device:R")
-		(at 198.12 215.9 90)
+		(at 208.28 215.9 90)
 		(unit 1)
 		(body_style 1)
@@
 		(dnp no)
 		(property "Reference" "R16"
-			(at 198.12 211.074 90)
+			(at 208.28 211.074 90)
 			(show_name no)
 			(do_not_autoplace no)
@@
 		)
 		(property "Value" "470R"
-			(at 198.12 213.614 90)
+			(at 208.28 213.614 90)
 			(show_name no)
 			(do_not_autoplace no)
@@
 		)
 		(property "Footprint" "Resistor_SMD:R_0603_1608Metric_Pad0.98x0.95mm_HandSolder"
-			(at 198.12 217.678 90)
+			(at 208.28 217.678 90)
 			(hide yes)
 			(show_name no)
@@
 		)
 		(property "Datasheet" ""
-			(at 198.12 215.9 0)
+			(at 208.28 215.9 0)
 			(hide yes)
 			(show_name no)
@@
 		)
 		(property "Description" "Resistor"
-			(at 198.12 215.9 0)
+			(at 208.28 215.9 0)
 			(hide yes)
 			(show_name no)
@@
 	(symbol
 		(lib_id "Device:R")
-		(at 198.12 205.74 90)
+		(at 208.28 205.74 90)
 		(unit 1)
 		(body_style 1)
@@
 		(dnp no)
 		(property "Reference" "R15"
-			(at 198.12 200.914 90)
+			(at 208.28 200.914 90)
 			(show_name no)
 			(do_not_autoplace no)
@@
 		)
 		(property "Value" "470R"
-			(at 198.12 203.454 90)
+			(at 208.28 203.454 90)
 			(show_name no)
 			(do_not_autoplace no)
@@
 		)
 		(property "Footprint" "Resistor_SMD:R_0603_1608Metric_Pad0.98x0.95mm_HandSolder"
-			(at 198.12 207.518 90)
+			(at 208.28 207.518 90)
 			(hide yes)
 			(show_name no)
@@
 		)
 		(property "Datasheet" ""
-			(at 198.12 205.74 0)
+			(at 208.28 205.74 0)
 			(hide yes)
 			(show_name no)
@@
 		)
 		(property "Description" "Resistor"
-			(at 198.12 205.74 0)
+			(at 208.28 205.74 0)
 			(hide yes)
 			(show_name no)

Commit message: almost done
Parts:
- D5, D6, D7: footprint LED_THT:LED_D5.0mm -> LED_THT:LED_D3.0mm
Connections:
- net at C28.2, C29.2: now also U10.3 (D); no longer J5.1 (Pin_1)
- net at J5.2 (Pin_2): now also U11.3 (D); no longer U10.3 (D)
- net at C28.1, R23.1: now also J5.1 (Pin_1); no longer U11.3 (D)
