File: driver1.kicad_pcb (KiCad board)
At the start: 2 copper layers, 84 parts, among them J1 FB CT, J2 GDT, J3 24VDC INPUT, U10 L7809, U11 L7805, U2 MCP6567, U4 IF-D95T, U6 TLV3501AID, U8 AOD609, U9 AOD609

Commit message: progress
Parts:
- removed C13: 100n, Capacitor_SMD:C_0603_1608Metric_Pad1.08x0.95mm_HandSolder
- added C29: 1u, Capacitor_SMD:C_1210_3225Metric_Pad1.33x2.70mm_HandSolder, F.Cu at (208.0, 76.3)
- added J4: PHASE, Connector_PinHeader_2.54mm:PinHeader_1x02_P2.54mm_Vertical_SMD_Pin1Left, F.Cu at (25.0, 82.5)
- added J5: GDT, TerminalBlock_Altech:Altech_AK100_1x02_P5.00mm, F.Cu at (211.4, 70.2)
- added R23: 15R, Resistor_SMD:R_1210_3225Metric_Pad1.30x2.65mm_HandSolder, F.Cu at (203.0, 76.3)
- added U1: L7809, Package_TO_SOT_SMD:TO-252-2, F.Cu at (73.5, 73.8)
- added U12: 74AHC158, Package_SO:TSSOP-16_4.4x5mm_P0.65mm, F.Cu at (25.8, 69.0)
- added U3: TLV3501AIDBV, Package_TO_SOT_SMD:SOT-23-6, F.Cu at (82.5, 40.6)
- added U5: IF-D95T, footprints:IF-D95T_IFB, F.Cu at (36.6, 59.0)
- added U7: 74AHC74, Package_SO:TSSOP-14_4.4x5mm_P0.65mm, F.Cu at (42.3, 74.1)
- C10, C3: value 100n -> 1n
- C11, C17: value 1u -> 100n
- C12, C6: value 10u -> 100n
- C15: value 10u -> 470u; footprint Capacitor_SMD:C_0603_1608Metric_Pad1.08x0.95mm_HandSolder -> Capacitor_THT:CP_Radial_D8.0mm_P3.50mm
- C16: value 4.7u -> 100n
- C18, C19: value 1000u -> 100n; footprint Capacitor_THT:CP_Radial_D12.5mm_P5.00mm -> Capacitor_SMD:C_0603_1608Metric_Pad1.08x0.95mm_HandSolder
- C2: value 1n -> 1000u; footprint Capacitor_SMD:C_0603_1608Metric_Pad1.08x0.95mm_HandSolder -> Capacitor_THT:CP_Radial_D12.5mm_P5.00mm
- C21: value 470u -> 1u; footprint Capacitor_THT:CP_Radial_D8.0mm_P3.50mm -> Capacitor_SMD:C_0805_2012Metric_Pad1.18x1.45mm_HandSolder
- C22, C26: value 100n -> 10u; footprint Capacitor_SMD:C_0603_1608Metric_Pad1.08x0.95mm_HandSolder -> Capacitor_SMD:C_0805_2012Metric_Pad1.18x1.45mm_HandSolder
- C23, C24: footprint Capacitor_SMD:C_0603_1608Metric_Pad1.08x0.95mm_HandSolder -> Capacitor_SMD:C_0805_2012Metric_Pad1.18x1.45mm_HandSolder
- C25: value 470u -> 10u; footprint Capacitor_THT:CP_Radial_D8.0mm_P3.50mm -> Capacitor_SMD:C_0805_2012Metric_Pad1.18x1.45mm_HandSolder
- C28: value 100n -> 4.7u; footprint Capacitor_SMD:C_0603_1608Metric_Pad1.08x0.95mm_HandSolder -> Capacitor_SMD:C_1210_3225Metric_Pad1.33x2.70mm_HandSolder
- C4: value 100n -> 1000u; footprint Capacitor_SMD:C_0603_1608Metric_Pad1.08x0.95mm_HandSolder -> Capacitor_THT:CP_Radial_D12.5mm_P5.00mm
- C8: value 1n -> 100n
- C9: value 100n -> 470u; footprint Capacitor_SMD:C_0603_1608Metric_Pad1.08x0.95mm_HandSolder -> Capacitor_THT:CP_Radial_D8.0mm_P3.50mm
- D1: value BAV99 -> BAT54SW; footprint Package_TO_SOT_SMD:SOT-23 -> Package_TO_SOT_SMD:SOT-323_SC-70
- D10: value SKIP -> 1N5819WS; footprint LED_THT:LED_D5.0mm -> Diode_SMD:D_SOD-323
- D2: value BAT54SW -> 1N5819WS; footprint Package_TO_SOT_SMD:SOT-323_SC-70 -> Diode_SMD:D_SOD-323
- D3: value 1N5819WS -> BAV99; footprint Diode_SMD:D_SOD-323 -> Package_TO_SOT_SMD:SOT-23
- D5: value 1N5819WS -> 5V_OK; footprint Diode_SMD:D_SOD-323 -> LED_THT:LED_D5.0mm
- D6: value 1N5819WS -> INTERRUPTER; footprint Diode_SMD:D_SOD-323 -> LED_THT:LED_D5.0mm
- D7: value 1N5819WS -> SKIP; footprint Diode_SMD:D_SOD-323 -> LED_THT:LED_D5.0mm
- D8: value 5V_OK -> 1N5819WS; footprint LED_THT:LED_D5.0mm -> Diode_SMD:D_SOD-323
- D9: value INTERRUPTER -> 1N5819WS; footprint LED_THT:LED_D5.0mm -> Diode_SMD:D_SOD-323
- H1, H2, H3, H4: value MountingHole -> MountingHole_Pad; footprint MountingHole:MountingHole_3.2mm_M3 -> MountingHole:MountingHole_3.2mm_M3_Pad
- J2: value GDT -> 24VDC INPUT
- J3: value 24VDC INPUT -> MODE; footprint TerminalBlock_Altech:Altech_AK100_1x02_P5.00mm -> Connector_PinHeader_2.54mm:PinHeader_1x03_P2.54mm_Vertical_SMD_Pin1Left
- R1: footprint Resistor_SMD:R_0603_1608Metric_Pad0.98x0.95mm_HandSolder -> Resistor_SMD:R_2512_6332Metric_Pad1.40x3.35mm_HandSolder
- R10, R6: value 1k -> 470R
- R11, R12, R17: value 1k -> 10k
- R14: value 2k -> 470R
- R15, R16: value 10k -> 470R
- R18: value 15R -> 1k
- R19, R20, R4: value 470R -> 10k
- R2: footprint Resistor_SMD:R_0603_1608Metric_Pad0.98x0.95mm_HandSolder -> Resistor_SMD:R_1210_3225Metric_Pad1.30x2.65mm_HandSolder
- R21, R3: value 470R -> 1k
- R22, R8: value 10k -> 1k
- R5: value 10k -> 2k
- RV1: footprint Potentiometer_THT:Potentiometer_Bourns_3339P_Vertical -> Potentiometer_THT:Potentiometer_Bourns_3296W_Vertical
- RV2: value 50k -> 10k
- RV4: value 10k -> 50k
- TP1: value OCD_ref -> UVLO_sense
- TP2: value UVLO_sense -> UVLO_ref
- TP3: value UVLO_ref -> OCD_ref
- U10: value L7809 -> AOD609; footprint Package_TO_SOT_SMD:TO-252-2 -> Package_TO_SOT_SMD:TO-252-4
- U11: value L7805 -> AOD609; footprint Package_TO_SOT_SMD:TO-252-2 -> Package_TO_SOT_SMD:TO-252-4
- U4: value IF-D95T -> L7805; footprint IF parts:IF-D95T_IFB -> Package_TO_SOT_SMD:TO-252-2
- U6: value TLV3501AID -> 74AHC14; footprint Package_SO:SOIC-8_3.9x4.9mm_P1.27mm -> Package_SO:TSSOP-14_4.4x5mm_P0.65mm
- U8: value AOD609 -> 74AHC1G08; footprint Package_TO_SOT_SMD:TO-252-4 -> Package_TO_SOT_SMD:SOT-353_SC-70-5
- U9: value AOD609 -> IX4340; footprint Package_TO_SOT_SMD:TO-252-4 -> Package_SO:SOIC-8-1EP_3.9x4.9mm_P1.27mm_EP2.29x3mm
- moved U9 144.3 mm to (25.3, 75.7)
- moved C21 130.6 mm to (35.5, 65.4)
- moved C25 130.5 mm to (35.5, 77.5)
- moved U6 126.6 mm to (42.3, 67.4)
- moved J1 116.2 mm to (24.6, 28.2)
- moved D4 115.6 mm to (79.2, 26.6)
- moved D2 115.5 mm to (79.2, 23.6)
- moved D5 112.3 mm to (69.0, 51.0)
- moved D3 111.5 mm to (57.9, 84.0)
- moved D6 110.3 mm to (69.0, 58.5)
- moved J3 110.0 mm to (25.0, 60.9)
- moved D7 108.4 mm to (69.0, 65.9)
- moved D1 107.3 mm to (30.9, 80.6)
- moved U2 105.6 mm to (51.2, 81.4)
- moved U8 104.0 mm to (62.3, 83.7)
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Connections:
- C10 pad 1: +5V -> Net-(D3-A)
- C10 pad 2: GND -> Net-(U3--)
- C11 pad 1: GND -> +24V
- C11 pad 2: +9V -> GND
- C12 pad 1: +24V -> GND
- C12 pad 2: GND -> +5V
- C14 pad 1: Net-(D5-A) -> +5V
- C14 pad 2: Net-(U1-OUTB) -> GND
- C15 pad 1: +24V -> +5V
- C16 pad 1: Net-(U8-D) -> GND
- C16 pad 2: Net-(J2-Pin_1) -> +5V
- C17 pad 1: Net-(C17-Pad1) -> +5V
- C17 pad 2: Net-(J2-Pin_1) -> GND
- C18 pad 1: +24V -> GND
- C18 pad 2: GND -> +5V
- C19 pad 1: +24V -> GND
- C19 pad 2: GND -> +5V
- C2 pad 1: Net-(D1-A) -> +24V
- C2 pad 2: Net-(U6--) -> GND
- C20 pad 1: +24V -> +5V
- C21 pad 1: +9V -> GND
- C21 pad 2: GND -> +9V
- C22 pad 1: +9V -> +5V
- C22 pad 2: GND -> Net-(D8-K)
- C23 pad 1: +24V -> Net-(D9-A)
- C23 pad 2: GND -> Net-(U10-G1)
- C24 pad 1: +5V -> Net-(D10-A)
- C24 pad 2: GND -> Net-(U11-G1)
- C25 pad 1: +5V -> +24V
- C26 pad 1: GND -> +24V
- C26 pad 2: +5V -> GND
- C27 pad 1: GND -> +5V
- C27 pad 2: +5V -> GND
- C28 pad 1: GND -> Net-(U10-D)
- C28 pad 2: +5V -> Net-(J5-Pin_1)
- C3 pad 1: GND -> Net-(U2B-+)
- C3 pad 2: +5V -> GND
- C4 pad 1: +5V -> +24V
- C5 pad 1: Net-(U2A-+) -> +24V
- C6 pad 1: +5V -> Net-(U2A-+)
- C6 pad 2: Net-(D3-K) -> GND
- C8 pad 1: Net-(U2B-+) -> +9V
- C9 pad 1: +5V -> +9V
- D1 pad 1: Net-(D1-A) -> GND
- D1 pad 2: Net-(D1-A) -> +5V
- D1 pad 3: GND -> Net-(D1-COM)
- D10 pad 1: GND -> +24V
- D2 pad 1: GND -> +24V
- D2 pad 2: +5V -> +9V
- D3 pad 1: Net-(D3-K) -> Net-(D3-A)
- D3 pad 2: GND -> Net-(D3-A)
- D4 pad 2: Net-(D4-A) -> +5V
- D5 pad 1: +24V -> GND
- D6 pad 1: +24V -> GND
- D6 pad 2: +9V -> Net-(D6-A)
- D7 pad 1: +24V -> GND
- D7 pad 2: +5V -> Net-(D7-A)
- D8 pad 1: GND -> Net-(D8-K)
- D8 pad 2: Net-(D8-A) -> GND
- D9 pad 1: GND -> +24V
- J2 pad 1: Net-(J2-Pin_1) -> GND
- J2 pad 2: Net-(J2-Pin_2) -> +24V
- J3 pad 1: GND -> INTERRUPTER
- J3 pad 2: +24V -> Net-(J3-Pin_2)
- R10 pad 1: Net-(D2-COM) -> Net-(U3-+)
- R10 pad 2: Net-(U2A--) -> Net-(C33-Pad1)
- R11 pad 1: ~{SKIP} -> Net-(U3--)
- R11 pad 2: +5V -> Net-(R11-Pad2)
- R12 pad 1: +24V -> Net-(U3-+)
- R12 pad 2: Net-(D4-A) -> FB
- R13 pad 1: +24V -> Net-(U5-OUTPUT)
- R13 pad 2: Net-(U2B-+) -> GND
- R14 pad 1: Net-(U2B-+) -> +5V
- R14 pad 2: GND -> Net-(D5-A)
- R15 pad 1: Net-(U4-OUTPUT) -> INTERRUPTER_LED
- R15 pad 2: GND -> Net-(D6-A)
- R16 pad 1: Net-(D3-K) -> SKIP_LED
- R16 pad 2: GND -> Net-(D7-A)
- R17 pad 1: +24V -> Net-(J3-Pin_2)
- R17 pad 2: Net-(D5-A) -> GND
- R18 pad 1: Net-(U8-D) -> ~{SKIP}
- R18 pad 2: Net-(C17-Pad1) -> +5V
- R19 pad 1: +5V -> Net-(D8-K)
- R19 pad 2: Net-(D8-A) -> GND
- R20 pad 1: INTERRUPTER_LED -> +5V
- R20 pad 2: Net-(D9-A) -> Net-(J4-Pin_1)
- R21 pad 1: SKIP_LED -> +24V
- R21 pad 2: Net-(D10-A) -> Net-(D9-A)
- R22 pad 1: +5V -> +24V
- R22 pad 2: Net-(SW1-B) -> Net-(D10-A)
- R3 pad 1: Net-(R3-Pad1) -> Net-(L1-Pad2)
- R3 pad 2: Net-(D1-A) -> Net-(D1-COM)
- R4 pad 1: Net-(U6-+) -> +24V
- R4 pad 2: Net-(C33-Pad1) -> Net-(U2B-+)
- R5 pad 1: Net-(U6-+) -> Net-(U2B-+)
- R5 pad 2: FB -> GND
- R6 pad 1: +5V -> Net-(R6-Pad1)
- R6 pad 2: Net-(U6-+) -> Net-(D3-A)
- R7 pad 1: Net-(U6-+) -> Net-(D1-COM)
- R7 pad 2: GND -> Net-(U2A--)
- R8 pad 1: Net-(U6--) -> +5V
- R8 pad 2: Net-(R8-Pad2) -> Net-(U3-+)
- R9 pad 1: Net-(L1-Pad2) -> Net-(U3-+)
- R9 pad 2: Net-(D2-COM) -> GND
- RV1 pad 2: Net-(R3-Pad1) -> Net-(R6-Pad1)
- RV2 pad 1: FB -> +5V
- RV2 pad 2: Net-(R8-Pad2) -> Net-(U2B--)
- RV2 pad 3: Net-(R8-Pad2) -> GND
- RV4 pad 1: +5V -> FB
- RV4 pad 2: Net-(U2B--) -> Net-(R11-Pad2)
- RV4 pad 3: GND -> Net-(R11-Pad2)
- TP1 pad 1: Net-(U2A-+) -> Net-(U2B-+)
- TP2 pad 1: Net-(U2B-+) -> Net-(U2B--)
- TP3 pad 1: Net-(U2B--) -> Net-(U2A-+)
- U10 pad 1: +24V -> GND
- U10 pad 2: GND -> Net-(U10-G1)
- U10 pad 3: +9V -> Net-(U10-D)
- U11 pad 1: +24V -> GND
- U11 pad 2: GND -> Net-(U11-G1)
- U11 pad 3: +5V -> Net-(J5-Pin_2)
- U4 pad 1: GND -> +24V
- U4 pad 2: Net-(U4-OUTPUT) -> GND
- U6 pad 1: unconnected-(U6-NC-Pad1) -> Net-(D8-K)
- U6 pad 2: Net-(U6--) -> ~{RESET}
- U6 pad 3: Net-(U6-+) -> Net-(U5-OUTPUT)
- U6 pad 4: GND -> Net-(U6-Pad4)
- U6 pad 5: unconnected-(U6-NC-Pad5) -> Net-(U6-Pad4)
- U6 pad 6: FB -> INTERRUPTER
- U6 pad 7: +5V -> GND
- U6 pad 8: GND -> INTERRUPTER_LED
- U8 pad 1: GND -> INTERRUPTER
- U8 pad 3: Net-(U8-D) -> GND
- U8 pad 4: +24V -> Net-(U7B-D)
- U8 pad 5: Net-(D4-A) -> +5V
- U9 pad 1: GND -> +9V
- U9 pad 2: Net-(U1-OUTB) -> A
- U9 pad 3: Net-(J2-Pin_2) -> GND
- U9 pad 4: +24V -> B
- U9 pad 5: Net-(D5-A) -> Net-(U11-G1)
Routing:
- net Net-(J5-Pin_2): track 0.00 -> 15.8 mm
- net Net-(U10-D): track 0.00 -> 2.12 mm
- added copper zone on F.Cu, net Net-(C29-Pad1)
- added copper zone on F.Cu, net Net-(J5-Pin_1)
- added copper zone on F.Cu, net Net-(U10-D)
Other:
- board outline added: 6.9 x 10.3 mm

Commit message: pcb progress
Parts:
- C11, C14, C18, C19, C20, C21, C25, C26, C27, C5, C8: moved to B.Cu
- J3: footprint Connector_PinHeader_2.54mm:PinHeader_1x03_P2.54mm_Vertical_SMD_Pin1Left -> Connector_PinHeader_2.54mm:PinHeader_1x03_P2.54mm_Vertical
- J4: footprint Connector_PinHeader_2.54mm:PinHeader_1x02_P2.54mm_Vertical_SMD_Pin1Left -> Connector_PinHeader_2.54mm:PinHeader_1x02_P2.54mm_Vertical
- U9: footprint Package_SO:SOIC-8-1EP_3.9x4.9mm_P1.27mm_EP2.29x3mm -> Package_SO:SOIC-8_3.9x4.9mm_P1.27mm
- moved H3 172.3 mm to (217.0, 115.0)
- moved H2 169.0 mm to (217.0, 25.0)
- moved C25 163.4 mm to (195.9, 46.5), turned to 90 degrees
- moved C26 162.5 mm to (195.9, 54.4), turned to 90 degrees
- moved U9 162.4 mm to (185.6, 50.1)
- moved C23 159.8 mm to (193.4, 47.1), turned to 90 degrees
- moved C24 159.1 mm to (193.4, 55.1), turned to 90 degrees
- moved C21 150.8 mm to (185.6, 50.7)
- moved U12 150.1 mm to (175.2, 54.4)
- moved C5 147.4 mm to (196.8, 36.2)
- moved C8 147.3 mm to (196.9, 40.8)
- moved J4 143.6 mm to (166.2, 56.4), turned to 180 degrees
- moved J3 136.5 mm to (161.1, 50.3), turned to 180 degrees
- moved U1 132.4 mm to (201.0, 38.5)
- moved U7 131.4 mm to (170.5, 45.3)
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Connections:
- C23 pad 2: Net-(U10-G1) -> Net-(U11-G1)
- C24 pad 2: Net-(U11-G1) -> Net-(U10-G1)
- C28 pad 1: Net-(U10-D) -> Net-(U11-D)
- R23 pad 1: Net-(U10-D) -> Net-(U11-D)
- U10 pad 3: Net-(U10-D) -> Net-(J5-Pin_2)
- U10 pad 5: Net-(D9-A) -> Net-(D10-A)
- U11 pad 3: Net-(J5-Pin_2) -> Net-(U11-D)
- U11 pad 5: Net-(D10-A) -> Net-(D9-A)
- U12 pad 10: GND -> Net-(U12-I0c)
- U12 pad 11: GND -> Net-(J4-Pin_1)
- U12 pad 12: unconnected-(U12-Zc-Pad12) -> A
- U12 pad 13: GND -> Net-(J4-Pin_1)
- U12 pad 14: GND -> Net-(U12-I0c)
- U12 pad 2: Net-(U12-I0a) -> GND
- U12 pad 3: Net-(J4-Pin_1) -> GND
- U12 pad 4: A -> unconnected-(U12-Za-Pad4)
- U12 pad 5: Net-(J4-Pin_1) -> GND
- U12 pad 6: Net-(U12-I0a) -> GND
- U12 pad 7: B -> unconnected-(U12-Zb-Pad7)
- U12 pad 9: unconnected-(U12-Zd-Pad9) -> B
- U6 pad 1: Net-(D8-K) -> Net-(U5-OUTPUT)
- U6 pad 10: Net-(U12-I0a) -> Net-(U12-I0c)
- U6 pad 12: unconnected-(U6-Pad12) -> ~{RESET}
- U6 pad 13: GND -> Net-(D8-K)
- U6 pad 2: ~{RESET} -> Net-(U6-Pad2)
- U6 pad 3: Net-(U5-OUTPUT) -> Net-(U6-Pad2)
- U6 pad 4: Net-(U6-Pad4) -> INTERRUPTER
- U6 pad 5: Net-(U6-Pad4) -> Net-(U6-Pad2)
- U6 pad 6: INTERRUPTER -> INTERRUPTER_LED
- U6 pad 8: INTERRUPTER_LED -> unconnected-(U6-Pad8)
- U6 pad 9: Net-(U6-Pad4) -> GND
- U8 pad 1: INTERRUPTER -> Net-(U7A-~{Q})
- U8 pad 2: Net-(U7A-~{Q}) -> INTERRUPTER
- U9 pad 5: Net-(U11-G1) -> Net-(U10-G1)
- U9 pad 7: Net-(U10-G1) -> Net-(U11-G1)
Routing:
- net ~{RESET}: track 0.00 -> 23.0 mm
- net Net-(U12-I0c): track 0.00 -> 20.1 mm, vias 0 -> 2
- net Net-(J4-Pin_1): track 0.00 -> 19.8 mm, vias 0 -> 2
- net INTERRUPTER: track 0.00 -> 14.8 mm
- net Net-(J3-Pin_2): track 0.00 -> 10.6 mm, vias 0 -> 1
- net Net-(D8-K): track 0.00 -> 10.1 mm
- net +24V: track 0.00 -> 9.56 mm, vias 0 -> 4
- net Net-(U7B-D): track 0.00 -> 9.05 mm, vias 0 -> 2
- net A: track 0.00 -> 8.79 mm
- net B: track 0.00 -> 8.34 mm
- net Net-(U12-E): track 0.00 -> 7.84 mm
- net FB: track 0.00 -> 7.70 mm
- net Net-(U11-G1): track 0.00 -> 6.72 mm
- net Net-(U10-G1): track 0.00 -> 6.20 mm
- net Net-(U7A-~{Q}): track 0.00 -> 4.35 mm
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- added copper zone on F.Cu, net +24V
- added copper zone on F.Cu, net +9V
- added copper zone on F.Cu, net Net-(D10-A)
- added copper zone on F.Cu, net Net-(D9-A)
- added copper zone on F.Cu, net Net-(J5-Pin_2)
- added copper zone on F.Cu, net Net-(U10-G1)
- added copper zone on F.Cu, net Net-(U11-G1)
- removed copper zone on F.Cu, net Net-(U10-D)
Other:
- board size 6.9 x 10.3 mm -> 100 x 100 mm

Commit message: baby steps
Parts:
- removed TP4: UVLO_out, TestPoint:TestPoint_Pad_D2.0mm
- C1, C12, C16, C17, C6, C7, R1, R13, R14, R15, R16, R17, R18, R20, R8, R9: moved to B.Cu
- moved C3 121.3 mm to (170.9, 29.4)
- moved C7 118.7 mm to (168.1, 24.4), turned to 90 degrees
- moved R5 117.9 mm to (170.9, 31.1)
- moved R4 117.4 mm to (170.9, 32.6), turned to 180 degrees
- moved D1 113.1 mm to (137.1, 41.6), turned to -90 degrees
- moved C12 107.6 mm to (156.8, 33.3), turned to -90 degrees
- moved RV2 106.8 mm to (166.3, 27.8), turned to -90 degrees
- moved U2 105.2 mm to (149.7, 44.1)
- moved RV4 104.8 mm to (158.1, 24.4)
- moved C33 102.5 mm to (156.5, 38.3), turned to 90 degrees
- moved R16 102.4 mm to (154.8, 68.4), turned to 90 degrees
- moved R13 100.4 mm to (157.6, 56.0)
- moved D3 100.3 mm to (142.7, 30.4)
- moved C16 98.5 mm to (150.6, 42.9)
- moved R8 98.5 mm to (156.5, 36.8), turned to -90 degrees
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Connections:
- C1 pad 1: Net-(J1-Pin_2) -> Net-(J1-Pin_1)
- D5 pad 1: GND -> Net-(D5-K)
- D5 pad 2: Net-(D5-A) -> +5V
- D6 pad 1: GND -> Net-(D6-K)
- D6 pad 2: Net-(D6-A) -> INTERRUPTER_LED
- D7 pad 1: GND -> Net-(D7-K)
- D7 pad 2: Net-(D7-A) -> SKIP_LED
- J1 pad 1: GND -> Net-(J1-Pin_1)
- J1 pad 2: Net-(J1-Pin_2) -> GND
- R1 pad 2: Net-(J1-Pin_2) -> Net-(J1-Pin_1)
- R14 pad 1: +5V -> Net-(D5-K)
- R14 pad 2: Net-(D5-A) -> GND
- R15 pad 1: INTERRUPTER_LED -> Net-(D6-K)
- R15 pad 2: Net-(D6-A) -> GND
- R16 pad 1: SKIP_LED -> Net-(D7-K)
- R16 pad 2: Net-(D7-A) -> GND
- RV1 pad 1: Net-(J1-Pin_2) -> Net-(J1-Pin_1)
Routing:
- net ~{RESET}: track 23.0 -> 0.00 mm
- net Net-(J1-Pin_1): track 0.00 -> 16.9 mm
- net Net-(L1-Pad1): track 0.00 -> 15.4 mm
- net Net-(U3-+): track 0.00 -> 8.68 mm, vias 0 -> 1
- net ~{SKIP}: track 0.00 -> 8.03 mm, vias 0 -> 1
- net Net-(L1-Pad2): track 0.00 -> 7.68 mm
- net +5V: track 0.00 -> 7.05 mm, vias 5 -> 7
- net Net-(D3-A): track 0.00 -> 5.36 mm
- net FB: track 7.70 -> 12.9 mm
- net GND: track 0.01 -> 4.76 mm, vias 83 -> 87
- net Net-(J4-Pin_1): track 19.8 -> 15.3 mm
- net Net-(D1-COM): track 0.00 -> 4.25 mm
- net Net-(R6-Pad1): track 0.00 -> 3.46 mm
- net Net-(D7-K): track 0.00 -> 2.09 mm
- net Net-(D6-K): track 0.00 -> 2.08 mm
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Other:
- board size 100 x 100 mm -> 99 x 100 mm

Commit message: almost done
Parts:
- D5, D6, D7: footprint LED_THT:LED_D5.0mm -> LED_THT:LED_D3.0mm
- moved H3 51.0 mm to (218.0, 64.0)
- moved H4 51.0 mm to (127.0, 64.0)
- moved RV3 12.6 mm to (143.8, 41.2), turned to 90 degrees
- moved U5 12.5 mm to (126.9, 51.6)
- moved R16 12.5 mm to (143.7, 62.7)
- moved C17 12.4 mm to (125.2, 53.5), turned to 90 degrees
- moved D7 12.1 mm to (142.0, 63.5)
- moved C6 11.6 mm to (145.5, 44.6), turned to -90 degrees
- moved RV4 9.40 mm to (148.7, 24.4)
- moved C16 7.64 mm to (157.7, 40.0)
- moved R18 7.64 mm to (161.1, 40.0)
- moved U2 7.64 mm to (156.7, 41.2)
- moved TP3 7.16 mm to (148.1, 47.2)
- moved R12 7.16 mm to (148.6, 34.6)
- moved R8 7.16 mm to (149.4, 35.5)
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Connections:
- C28 pad 1: Net-(U11-D) -> Net-(J5-Pin_1)
- C28 pad 2: Net-(J5-Pin_1) -> Net-(U10-D)
- C29 pad 2: Net-(J5-Pin_1) -> Net-(U10-D)
- R23 pad 1: Net-(U11-D) -> Net-(J5-Pin_1)
- U10 pad 3: Net-(J5-Pin_2) -> Net-(U10-D)
- U11 pad 3: Net-(U11-D) -> Net-(J5-Pin_2)
Routing:
- net FB: track 12.9 -> 53.8 mm, vias 0 -> 1
- net Net-(U5-OUTPUT): track 0.00 -> 30.6 mm
- net ~{RESET}: track 0.00 -> 22.9 mm
- net Net-(U2B--): track 1.70 -> 21.8 mm
- net Net-(U2B-+): track 0.00 -> 18.1 mm
- net Net-(U2A--): track 0.00 -> 15.3 mm
- net ~{SKIP}: track 8.03 -> 21.7 mm, vias 1 -> 2
- net Net-(U2A-+): track 1.70 -> 13.4 mm
- net Net-(U3--): track 0.00 -> 8.49 mm
- net Net-(J3-Pin_2): track 9.85 -> 1.67 mm
- net Net-(R11-Pad2): track 0.00 -> 6.84 mm
- net Net-(J4-Pin_1): track 15.3 -> 20.7 mm
- net +24V: track 9.56 -> 14.2 mm
- net Net-(U7B-D): track 9.05 -> 13.3 mm, vias 2 -> 0
- net Net-(J5-Pin_2): track 17.9 -> 15.8 mm
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- added copper zone on F.Cu, net +5V
- added copper zone on B.Cu, net GND
- added copper zone on F.Cu, net Net-(U10-D)
- removed copper zone on F.Cu, net Net-(J5-Pin_2)

Commit message: infant steps
Parts:
- moved TP3 2.75 mm to (148.1, 44.5)
Routing:
- net SKIP_LED: track 0.00 -> 31.9 mm
- net Net-(J3-Pin_2): track 1.67 -> 15.3 mm
- net INTERRUPTER_LED: track 0.00 -> 10.6 mm
- net Net-(U2A-+): track 13.4 -> 17.9 mm
- net Net-(U12-I0c): track 17.5 -> 20.6 mm, vias 0 -> 2
- net Net-(D7-K): track 0.00 -> 1.72 mm
- net Net-(D6-K): track 0.00 -> 1.72 mm
- net Net-(D5-K): track 0.00 -> 1.71 mm
- net GND: vias 94 -> 95
Other:
- board size 99 x 100 mm -> 99 x 48 mm
- board text added: "todo: - move ct connector to top side - shrink - fix silkscreen - add labels maybe - f gnd outline"
Changed lines of the file:
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@@
 			)
 		)
-		(clearance 2.5)
+		(clearance 1)
 		(attr exclude_from_bom)
 		(duplicate_pad_numbers_are_jumpers no)
@@
 	(footprint "TestPoint:TestPoint_Pad_D2.0mm"
 		(layer "F.Cu")
-		(at 148.1 47.2)
+		(at 148.05 44.45)
 		(descr "SMD pad as test Point, diameter 2.0mm")
 		(tags "test point SMD pad")
@@
 			)
 		)
-		(clearance 2.5)
+		(clearance 1)
 		(attr exclude_from_bom)
 		(duplicate_pad_numbers_are_jumpers no)
@@
 			)
 		)
-		(clearance 2.5)
+		(clearance 1)
 		(attr exclude_from_bom)
 		(duplicate_pad_numbers_are_jumpers no)
@@
 			)
 		)
-		(clearance 2.5)
+		(clearance 1)
 		(attr exclude_from_bom)
 		(duplicate_pad_numbers_are_jumpers no)
@@
 	(gr_rect
 		(start 122.981272 19.984416)
-		(end 221.981272 119.984416)
+		(end 221.981272 67.984416)
 		(stroke
 			(width 0.05)
-			(type default)
+			(type solid)
 		)
 		(fill no)
 		(layer "Edge.Cuts")
 	)
+	(gr_text "todo:\n- move ct connector to top side\n- shrink\n- fix silkscreen\n- add labels maybe\n- f gnd outline"
+		(at 242 36 0)
+		(layer "User.1")
+		(effects
+			(font
+				(size 1 1)
+				(thickness 0.15)
+			)
+			(justify left bottom)
+		)
+	)
 	(via
 		(at 156.45 56.2475)
@@
 	)
 	(segment
+		(start 146.501332 60.987395)
+		(end 147.991227 59.4975)
+		(width 0.2)
+		(layer "F.Cu")
+		(net "INTERRUPTER_LED")
+	)
+	(segment
+		(start 147.991227 59.4975)
+		(end 156.45 59.4975)
+		(width 0.2)
+		(layer "F.Cu")
+		(net "INTERRUPTER_LED")
+	)
+	(segment
 		(start 171.675 55.39)
 		(end 171.6675 55.3975)
@@
 	)
 	(via
+		(at 163.4625 50.55)
+		(size 0.4)
+		(drill 0.2)
+		(layers "F.Cu" "B.Cu")
+		(net "GND")
+	)
+	(via
 		(at 201.717909 39)
 		(size 0.6)
@@
 		(net "Net-(U12-I0c)")
 	)
+	(via
+		(at 178.0125 53.44)
+		(size 0.4)
+		(drill 0.2)
+		(layers "F.Cu" "B.Cu")
+		(net "Net-(U12-I0c)")
+	)
+	(via
+		(at 178.0125 56.04)
+		(size 0.4)
+		(drill 0.2)
+		(layers "F.Cu" "B.Cu")
+		(net "Net-(U12-I0c)")
+	)
+	(segment
+		(start 178.0125 56.04)
+		(end 177.955393 56.04)
+		(width 0.2)
+		(layer "B.Cu")
+		(net "Net-(U12-I0c)")
+	)
+	(segment
+		(start 177.5125 55.597107)
+		(end 177.5125 53.882893)
+		(width 0.2)
+		(layer "B.Cu")
+		(net "Net-(U12-I0c)")
+	)
+	(segment
+		(start 177.955393 56.04)
+		(end 177.5125 55.597107)
+		(width 0.2)
+		(layer "B.Cu")
+		(net "Net-(U12-I0c)")
+	)
+	(segment
+		(start 177.955393 53.44)
+		(end 178.0125 53.44)
+		(width 0.2)
+		(layer "B.Cu")
+		(net "Net-(U12-I0c)")
+	)
+	(segment
+		(start 177.5125 53.882893)
+		(end 177.955393 53.44)
+		(width 0.2)
+		(layer "B.Cu")
+		(net "Net-(U12-I0c)")
+	)
 	(segment
 		(start 173.249044 58.1975)
@@
 	)
 	(segment
+		(start 144.55 44.45)
+		(end 143.8 43.7)
+		(width 0.2)
+		(layer "F.Cu")
+		(net "Net-(U2A-+)")
+	)
+	(segment
+		(start 148.05 44.45)
+		(end 144.55 44.45)
+		(width 0.2)
+		(layer "F.Cu")
+		(net "Net-(U2A-+)")
+	)
+	(segment
 		(start 143.8 43.7)
 		(end 145.975 41.525)
@@
 	)
 	(segment
+		(start 165.869817 43.634816)
+		(end 166.900001 44.665)
+		(width 0.2)
+		(layer "B.Cu")
+		(net "Net-(J3-Pin_2)")
+	)
+	(segment
+		(start 159.317276 47.324816)
+		(end 158.167276 46.174816)
+		(width 0.2)
+		(layer "B.Cu")
+		(net "Net-(J3-Pin_2)")
+	)
+	(segment
+		(start 158.167276 46.174816)
+		(end 158.167276 44.30847)
+		(width 0.2)
+		(layer "B.Cu")
+		(net "Net-(J3-Pin_2)")
+	)
+	(segment
+		(start 166.900001 44.665)
+		(end 167.6375 44.665)
+		(width 0.2)
+		(layer "B.Cu")
+		(net "Net-(J3-Pin_2)")
+	)
+	(segment
+		(start 158.84093 43.634816)
+		(end 165.869817 43.634816)
+		(width 0.2)
+		(layer "B.Cu")
+		(net "Net-(J3-Pin_2)")
+	)
+	(segment
 		(start 167.6375 44.665)
 		(end 168.9475 44.665)
@@
 	)
 	(segment
+		(start 158.167276 44.30847)
+		(end 158.84093 43.634816)
+		(width 0.2)
+		(layer "B.Cu")
+		(net "Net-(J3-Pin_2)")
+	)
+	(segment
 		(start 172.625001 45.315)
 		(end 172.2875 45.652501)
@@
 	)
 	(segment
+		(start 137.501332 63.527395)
+		(end 139.171332 63.527395)
+		(width 0.2)
+		(layer "B.Cu")
+		(net "Net-(D5-K)")
+	)
+	(segment
+		(start 139.171332 63.527395)
+		(end 139.201332 63.557395)
+		(width 0.2)
+		(layer "B.Cu")
+		(net "Net-(D5-K)")
+	)
+	(segment
 		(start 166.0975 46.615)
 		(end 167.6375 46.615)
@@
 	)
 	(segment
+		(start 142.001332 63.527395)
+		(end 143.658832 63.527395)
+		(width 0.2)
+		(layer "B.Cu")
+		(net "Net-(D7-K)")
+	)
+	(segment
+		(start 143.658832 63.527395)
+		(end 143.701332 63.569895)
+		(width 0.2)
+		(layer "B.Cu")
+		(net "Net-(D7-K)")
+	)
+	(segment
+		(start 157.023727 45.965)
+		(end 167.6375 45.965)
+		(width 0.2)
+		(layer "F.Cu")
+		(net "SKIP_LED")
+	)
+	(segment
+		(start 142.001332 60.987395)
+		(end 157.023727 45.965)
+		(width 0.2)
+		(layer "F.Cu")
+		(net "SKIP_LED")
+	)
+	(segment
 		(start 159.624999 41.525)
 		(end 165.2 35.949999)
@@
 	)
 	(segment
+		(start 146.501332 63.527395)
+		(end 148.158832 63.527395)
+		(width 0.2)
+		(layer "B.Cu")
+		(net "Net-(D6-K)")
+	)
+	(segment
+		(start 148.158832 63.527395)
+		(end 148.201332 63.569895)
+		(width 0.2)
+		(layer "B.Cu")
+		(net "Net-(D6-K)")
+	)
+	(segment

Commit message: the wheels on the bus go round and round
Parts:
- moved RV1 58.7 mm to (79.3, 37.6)
- moved RV3 58.7 mm to (85.3, 46.4)
- moved TP3 58.7 mm to (89.5, 49.6)
- moved C10 58.7 mm to (84.5, 39.2)
- moved C6 58.7 mm to (87.0, 49.8)
- moved D1 58.7 mm to (78.6, 46.8)
- moved L1 58.7 mm to (67.0, 49.7)
- moved R1 58.7 mm to (73.0, 40.6)
- moved R10 58.7 mm to (89.4, 42.2)
- moved R12 58.7 mm to (90.1, 39.8)
- moved R2 58.7 mm to (75.6, 48.1)
- moved R3 58.7 mm to (79.0, 49.7)
- moved R6 58.7 mm to (82.9, 39.2)
- moved R7 58.7 mm to (81.5, 48.8)
- moved R9 58.7 mm to (89.4, 40.7)
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Routing:
- net SKIP_LED: track 31.9 -> 0.00 mm
- net Net-(U5-OUTPUT): track 30.6 -> 0.00 mm, vias 1 -> 0
- net FB: track 53.8 -> 37.4 mm
- net Net-(J1-Pin_1): track 16.9 -> 3.03 mm
- net Net-(U2B-+): track 18.1 -> 5.04 mm
- net Net-(U2B--): track 21.8 -> 8.97 mm
- net ~{SKIP}: track 21.7 -> 9.81 mm
- net INTERRUPTER_LED: track 10.6 -> 0.00 mm
- net Net-(U2A--): track 15.3 -> 6.28 mm
- net Net-(U2A-+): track 17.9 -> 9.33 mm
- net GND: vias 95 -> 409
- added copper zone on F.Cu, net GND
Other:
- board size 99 x 48 mm -> 96 x 48 mm
- board text added: "todo: - put shit back - fix silkscreen - add labels maybe"
- board text removed: "todo: - move ct connector to top side - shrink - fix silkscreen - add labels maybe - f gnd outline"

Commit message: i hate zones
Parts:
- moved RV1 71.9 mm to (149.8, 23.7)
- moved RV4 69.5 mm to (159.7, 28.8), turned to -90 degrees
- moved R1 69.1 mm to (141.0, 28.4), turned to 0 degrees
- moved R11 67.1 mm to (154.9, 26.1), turned to 0 degrees
- moved L1 66.9 mm to (131.4, 31.9), turned to -90 degrees
- moved D1 65.8 mm to (142.8, 32.2), turned to 180 degrees
- moved C10 65.7 mm to (149.9, 33.2), turned to 90 degrees
- moved R6 65.7 mm to (148.3, 33.2), turned to -90 degrees
- moved C6 65.3 mm to (151.9, 42.6), turned to 0 degrees
- moved R12 65.0 mm to (154.7, 32.3)
- moved R9 65.0 mm to (154.0, 33.2)
- moved C12 65.0 mm to (155.8, 29.8)
- moved C33 65.0 mm to (155.5, 34.7)
- moved R8 65.0 mm to (155.5, 33.2)
- moved R10 65.0 mm to (154.0, 34.7)
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Routing:
- net SKIP_LED: track 0.00 -> 30.5 mm
- net Net-(U5-OUTPUT): track 0.00 -> 29.1 mm, vias 0 -> 1
- net ~{SKIP}: track 9.81 -> 20.2 mm
- net Net-(J1-Pin_1): track 3.03 -> 12.9 mm
- net Net-(U2A--): track 6.28 -> 16.0 mm
- net Net-(U2B-+): track 5.04 -> 14.8 mm
- net Net-(U2B--): track 8.97 -> 18.1 mm
- net INTERRUPTER_LED: track 0.00 -> 8.14 mm
- net +24V: track 14.2 -> 22.1 mm
- net FB: track 37.4 -> 43.7 mm
- net Net-(L1-Pad1): track 15.4 -> 20.0 mm, vias 0 -> 1
- net Net-(U2A-+): track 9.33 -> 13.8 mm
- net Net-(R6-Pad1): track 3.46 -> 7.58 mm
- net Net-(L1-Pad2): track 7.68 -> 9.56 mm
- net Net-(D1-COM): track 4.25 -> 3.73 mm
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Other:
- board text added: "todo: - add labels maybe"
- board text removed: "todo: - put shit back - fix silkscreen - add labels maybe"
